File: Costruzione VFO ESP32/kicad/schema-vf0-retro-scala-esp32/schema-vf0-retro-scala-esp32.kicad_sch (KiCad schematic)
At the start: 24 parts, among them J1 Conn_01x15_Pin, J2 Conn_01x15_Pin, J3 SI5351, J4 ST7735, Q1 NPN, SW1 STORE RED, SW2 MEM-CH, SW3 RIT, SW4 STEP+, SW5 STEP-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

Commit message: update
Parts:
- R7: value 2K2 -> 220
Connections:
- net D16 is gone; now on net D16-ENCB: J1.10 (Pin_10)
- net D17 is gone; now on net D17-ENCA: J1.9 (Pin_9)
- net D21 is gone; now on net D21-SDA: J1.5 (Pin_5)
- net D22 is gone; now on net D22-SCL: J1.2 (Pin_2)
- net D25 is gone; now on net D25-MEM: J2.8 (Pin_8)
- net D26 is gone; now on net D26-ST+: J2.9 (Pin_9)
- net D27 is gone; now on net D27-ST-: J2.10 (Pin_10)
- net D32 is gone; now on net D32-STO: J2.6 (Pin_6)
- net D33 is gone; now on net D33-TX/: J2.7 (Pin_7)
- net DXX-AUX is gone; now on net D14-AUX: SW6.3 (C)
- net DXX-RIT is gone; now on net D18-RIT: SW3.3 (C)
- net DXX-RITON is gone; now on net D19-LEDRIT: R7.1
- net D12 renamed D12-boot mode
- net D13 renamed D13-flash
- net D14 renamed D14-AUX
- net D18 renamed D18-RIT
- net D19 renamed D19-LEDRIT
- net D34 renamed D34-POTRIT
